Commit message: Stabilize Spot collision IK from bundled assets
Update the bundled Spot collision geometry to match the reference IK behavior while preserving the previous visual meshes, remove the temporary solver-side collision workaround, expose collision-geometry inspection in the Viser example, and include the auxiliary body boxes in the curated distal-arm collision set.

Constraint: Main should receive the Spot work as one squashed feature commit.

Rejected: Keeping the ad hoc collision workaround | the packaged collision asset and curated pair list now reproduce the intended behavior directly.

Rejected: Enabling all body-arm collision pairs | curated distal-arm/body-box pairs cover the observed gap with less solver/debug noise.

Confidence: high

Scope-risk: moderate

Directive: Preserve visual meshes unless intentionally changing appearance; validate Spot collision changes with the packaged URDF headless regression before modifying curated pairs.

Tested: pixi run pytest -q test/test_spot_whole_body_ik_headless.py; python3 -m py_compile examples/14_spot_full_body_ik_viser.py examples/example_helpers/spot_whole_body_ik.py test/test_spot_whole_body_ik_headless.py; git diff --check --cached.

Not-tested: Manual browser manipulation against the collision geometry after squashing to main.

File: examples/assets/spot_description/urdf/spot_with_arm.urdf (robot description, URDF)
Before this commit: robot spot, 28 links, 27 joints
Links:
- removed link arm_link_el0
- removed link arm_link_el1
- removed link arm_link_fngr
- removed link arm_link_hr0
- removed link arm_link_sh0
- removed link arm_link_sh1
- removed link arm_link_wr0
- removed link arm_link_wr1
- removed link base_link
- removed link front_left_foot
- removed link front_left_hip
- removed link front_left_lower_leg
- removed link front_left_upper_leg
- removed link front_rail
- removed link front_right_foot
- removed link front_right_hip
- removed link front_right_lower_leg
- removed link front_right_upper_leg
- removed link rear_left_foot
- removed link rear_left_hip
- removed link rear_left_lower_leg
- removed link rear_left_upper_leg
- removed link rear_rail
- removed link rear_right_foot
- removed link rear_right_hip
- removed link rear_right_lower_leg
- removed link rear_right_upper_leg
- added link arm0_link_el0, mass 0.94831958; collision mesh filename=../meshes/arm/collision/arm_link_el0.obj; visual mesh filename=../meshes/arm/visual/arm_link_el0.obj
- added link arm0_link_el1, mass 1.01754820; collision mesh filename=../meshes/arm/collision/arm_link_el1_lip.obj; collision mesh filename=../meshes/arm/collision/arm_link_el1_main.obj
- added link arm0_link_fngr, mass 0.22383315; collision mesh filename=../meshes/gripper/collision/left_finger.obj; collision mesh filename=../meshes/gripper/collision/left_hinge.obj
- added link arm0_link_jaw; collision mesh filename=../meshes/gripper/collision/front_jaw.obj; collision mesh filename=../meshes/gripper/collision/jaw_tooth.obj
- added link arm0_link_sh0, mass 1.904699; collision mesh filename=../meshes/arm/collision/arm_link_sh0_base.obj; collision mesh filename=../meshes/arm/collision/arm_link_sh0_left_motor.obj
- added link arm0_link_sh1, mass 1.85701942; collision mesh filename=../meshes/arm/collision/arm_link_sh1.obj; visual mesh filename=../meshes/arm/visual/arm_link_sh1.obj
- added link arm0_link_wr0, mass 0.58263740; collision mesh filename=../meshes/arm/collision/arm_link_wr0.obj; visual mesh filename=../meshes/arm/visual/arm_link_wr0.obj
- added link arm0_link_wr1, mass 0.93335298; collision mesh filename=../meshes/arm/collision/arm_link_wr1.obj; visual mesh filename=../meshes/arm/visual/arm_link_wr1.obj
- added link base
- added link fl_foot; collision sphere radius=0.035
- added link fl_hip, mass 1.13688339; visual mesh filename=../meshes/base/visual/front_left_hip.obj
- added link fl_lleg, mass 0.330; collision mesh filename=../meshes/base/collision/lower_leg_collision.obj; visual mesh filename=../meshes/base/visual/front_left_lower_leg.obj
- added link fl_uleg, mass 2.25620359; collision mesh filename=../meshes/base/collision/upper_leg_collision.obj; visual mesh filename=../meshes/base/visual/front_left_upper_leg.obj
- added link fr_foot; collision sphere radius=0.035
- added link fr_hip, mass 1.13688339; visual mesh filename=../meshes/base/visual/front_right_hip.obj
- added link fr_lleg, mass 0.330; collision mesh filename=../meshes/base/collision/lower_leg_collision.obj; visual mesh filename=../meshes/base/visual/front_right_lower_leg.obj
- added link fr_uleg, mass 2.25620359; collision mesh filename=../meshes/base/collision/upper_leg_collision.obj; visual mesh filename=../meshes/base/visual/front_right_upper_leg.obj
- added link hl_foot; collision sphere radius=0.035
- added link hl_hip, mass 1.13688339; visual mesh filename=../meshes/base/visual/rear_left_hip.obj
- added link hl_lleg, mass 0.330; collision mesh filename=../meshes/base/collision/lower_leg_collision.obj; visual mesh filename=../meshes/base/visual/rear_left_lower_leg.obj
- added link hl_uleg, mass 2.25620359; collision mesh filename=../meshes/base/collision/upper_leg_collision.obj; visual mesh filename=../meshes/base/visual/rear_left_upper_leg.obj
- added link hr_foot; collision sphere radius=0.035
- added link hr_hip, mass 1.13688339; visual mesh filename=../meshes/base/visual/rear_right_hip.obj
- added link hr_lleg, mass 0.330; collision mesh filename=../meshes/base/collision/lower_leg_collision.obj; visual mesh filename=../meshes/base/visual/rear_right_lower_leg.obj
- added link hr_uleg, mass 2.25620359; collision mesh filename=../meshes/base/collision/upper_leg_collision.obj; visual mesh filename=../meshes/base/visual/rear_right_upper_leg.obj
- link body: mass None -> 16.70765207; geometry collision box size=0.045 0.18 0.18; collision box size=0.065 0.16 0.145
Joints:
- removed joint arm_el0
- removed joint arm_el1
- removed joint arm_f1x
- removed joint arm_hr0
- removed joint arm_sh0
- removed joint arm_sh1
- removed joint arm_wr0
- removed joint arm_wr1
- removed joint base_link_joint
- removed joint front_left_ankle
- removed joint front_left_hip_x
- removed joint front_left_hip_y
- removed joint front_left_knee
- removed joint front_rail_joint
- removed joint front_right_ankle
- removed joint front_right_hip_x
- removed joint front_right_hip_y
- removed joint front_right_knee
- removed joint rear_left_ankle
- removed joint rear_left_hip_x
- removed joint rear_left_hip_y
- removed joint rear_left_knee
- removed joint rear_rail_joint
- removed joint rear_right_ankle
- removed joint rear_right_hip_x
- removed joint rear_right_hip_y
- removed joint rear_right_knee
- added joint arm0_el0: type revolute, parent arm0_link_sh1, child arm0_link_el0, origin xyz=0.3385 0 0 rpy=0 0 0, axis 0 1 0, limit lower=0 upper=3.14159 effort=90.9 velocity=999
- added joint arm0_el1: type revolute, parent arm0_link_el0, child arm0_link_el1, origin xyz=0.40330 0.0 0.0750 rpy=0 0 0, axis 1 0 0, limit lower=-2.792530 upper=2.792530 effort=30.3 velocity=999
- added joint arm0_f1x: type revolute, parent arm0_link_wr1, child arm0_link_fngr, origin xyz=0.11745 0.0 0.014820 rpy=0 0 0, axis 0.0 1.0 0.0, limit lower=-1.5708 upper=0.0 effort=15.32 velocity=999
- added joint arm0_jaw: type fixed, parent arm0_link_wr1, child arm0_link_jaw
- added joint arm0_sh0: type revolute, parent body, child arm0_link_sh0, origin xyz=0.292 0.0 0.188 rpy=0 0 0, axis 0 0 1, limit lower=-2.61799 upper=3.14159 effort=90.9 velocity=999
- added joint arm0_sh1: type revolute, parent arm0_link_sh0, child arm0_link_sh1, origin xyz=0.0 0.0 0.0 rpy=0 0 0, axis 0 1 0, limit lower=-3.14159 upper=0.523599 effort=181.8 velocity=999
- added joint arm0_wr0: type revolute, parent arm0_link_el1, child arm0_link_wr0, origin xyz=0.0 0.0 0.0 rpy=0 0 0, axis 0 1 0, limit lower=-1.8326 upper=1.8326 effort=30.3 velocity=999
- added joint arm0_wr1: type revolute, parent arm0_link_wr0, child arm0_link_wr1, origin xyz=0.0 0.0 0.0 rpy=0 0 0, axis 1 0 0, limit lower=-2.87989 upper=2.87979 effort=30.3 velocity=999
- added joint base_virtual_joint: type fixed, parent base, child body
- added joint fl_ank: type fixed, parent fl_lleg, child fl_foot, origin xyz=0.0 0.0 -0.3365
- added joint fl_hx: type revolute, parent body, child fl_hip, origin xyz=0.29785 0.05500 0.00000 rpy=0 0 0, axis 1 0 0, limit lower=-0.785398 upper=0.785398 effort=45 velocity=100
- added joint fl_hy: type revolute, parent fl_hip, child fl_uleg, origin xyz=0.0 0.110945 0.0 rpy=0 0 0, axis 0 1 0, limit lower=-0.898845 upper=2.295108 effort=45 velocity=100
- added joint fl_kn: type revolute, parent fl_uleg, child fl_lleg, origin xyz=0.025 0.000 -0.3205 rpy=0 0 0, axis 0 1 0, limit lower=-2.7929 upper=-0.2471 effort=115 velocity=100
- added joint fr_ank: type fixed, parent fr_lleg, child fr_foot, origin xyz=0.0 0.0 -0.3365
- added joint fr_hx: type revolute, parent body, child fr_hip, origin xyz=0.29785 -0.05500 0.00000 rpy=0 0 0, axis 1 0 0, limit lower=-0.785398 upper=0.785398 effort=45 velocity=100
- added joint fr_hy: type revolute, parent fr_hip, child fr_uleg, origin xyz=0.0 -0.110945 0.0 rpy=0 0 0, axis 0 1 0, limit lower=-0.898845 upper=2.295108 effort=45 velocity=100
- added joint fr_kn: type revolute, parent fr_uleg, child fr_lleg, origin xyz=0.025 0.000 -0.3205 rpy=0 0 0, axis 0 1 0, limit lower=-2.7929 upper=-0.2471 effort=115 velocity=100
- added joint hl_ank: type fixed, parent hl_lleg, child hl_foot, origin xyz=0.0 0.0 -0.3365
- added joint hl_hx: type revolute, parent body, child hl_hip, origin xyz=-0.29785 0.05500 0.00000 rpy=0 0 0, axis 1 0 0, limit lower=-0.785398 upper=0.785398 effort=45 velocity=100
- added joint hl_hy: type revolute, parent hl_hip, child hl_uleg, origin xyz=0.0 0.110945 0.0 rpy=0 0 0, axis 0 1 0, limit lower=-0.898845 upper=2.295108 effort=45 velocity=100
- added joint hl_kn: type revolute, parent hl_uleg, child hl_lleg, origin xyz=0.025 0.000 -0.3205 rpy=0 0 0, axis 0 1 0, limit lower=-2.7929 upper=-0.2471 effort=115 velocity=100
- added joint hr_ank: type fixed, parent hr_lleg, child hr_foot, origin xyz=0.0 0.0 -0.3365
- added joint hr_hx: type revolute, parent body, child hr_hip, origin xyz=-0.29785 -0.05500 0.00000 rpy=0 0 0, axis 1 0 0, limit lower=-0.785398 upper=0.785398 effort=45 velocity=100
- added joint hr_hy: type revolute, parent hr_hip, child hr_uleg, origin xyz=0.0 -0.110945 0.0 rpy=0 0 0, axis 0 1 0, limit lower=-0.898845 upper=2.295108 effort=45 velocity=100
- added joint hr_kn: type revolute, parent hr_uleg, child hr_lleg, origin xyz=0.025 0.000 -0.3205 rpy=0 0 0, axis 0 1 0, limit lower=-2.7929 upper=-0.2471 effort=115 velocity=100
